File: hardware/cape/holobone.sch (KiCad schematic (older format))
At the start: 10 parts, among them P8 BeagleBone_Black_Header, P9 BeagleBone_Black_Header

Commit message: add schematics
Parts:
- added C1, C2: 0.1uF, symbol Device:C_Small
- added C10: 100 nF, symbol Device:C_Small
- added C11: 2.2 uF, symbol Device:C_Small
- added C3, C5: 1uF, symbol Device:C_Small
- added C6: 10uF, symbol Device:C_Small
- added C7: 3.3uF, symbol Device:C_Small
- added C8: 22nF, symbol Device:C_Small
- added C9: 1000 pF, symbol Device:C_Small
- added J1, J2, J3, J4: Conn_01x03, symbol Connector_Generic:Conn_01x03
- added L1: 47 uH, symbol Device:L
- added R10, R11, R12, R13, R16, R17, R5, R7: 16.9k, symbol Device:R_Small
- added R18: 4.7M, symbol Device:R_Small
- added R19: 10 k, symbol Device:R_Small
- added R20: R, symbol Device:R_Small
- added R21: 10R, symbol Device:R_Small
- added R22: 147 k, symbol Device:R_Small
- added R23: 28 k, symbol Device:R_Small
- added R4, R6: 4.12k, symbol Device:R_Small
- added R8, R9: 11.3k, symbol Device:R_Small
- added U1: MAX5137GTG+, symbol holobone:MAX5137GTG+
- added U2, U3: TL084, symbol Amplifier_Operational:TL084
- added U5: MCP1804x-5002xOT, Package_TO_SOT_SMD:SOT-23-5, symbol Regulator_Linear:MCP1804x-5002xOT
- added U6: ST1S50, symbol holobone:ST1S50
- gave numbers to parts that had none: 8
Connections:
- net +3V3: now also C1.2, R20.1, U1.3 (DVDD)
- net +5V: now also C11.2, L1.2, R22.1
- net GND: now also C2.1, C3.1, C5.1, C6.1, J1.2 (Pin_2), J2.2 (Pin_2), J3.2 (Pin_2), R8.2, R9.2, U1.19 (AGND), U1.21 (REFO), U1.22 (REFI), U1.7 (AGND), U2.10 (+), U2.3 (+), U3.10 (+), U5.2 (GND), U6.1 (GNDP); no longer C4.2, U4.4 (GND)
- net GNDD: now also C4.2, U4.4 (GND), C1.1, C11.1, C7.1, C8.1, C9.1, J4.2 (Pin_2), R18.2, R23.2, U6.4 (GNDA)
- net SCL: now also P9.19 (Pin_19)
- net SDA: now also P9.20 (Pin_20)
- net CS_DAC: now reaches P9.17 (Pin_17)
- net CS_DAC: now also U1.10 (~CS)
- net SCLK: now reaches P9.22 (Pin_22)
- net SCLK: now also U1.12 (SCLK)
- net POWER_GOOD: now reaches P9.29 (Pin_29)
- net POWER_GOOD: now also R20.2, U6.8 (PG)
- net MOSI: now reaches P9.30 (Pin_30)
- net MOSI: now also U1.9 (DIN)
- net LDAC: now reaches P9.31 (Pin_31)
- net LDAC: now also U1.15 (~LDAC)
- net AUX0: now reaches P8.45 (Pin_45)
- net AUX0: now also J4.1 (Pin_1)
- net AUX1: now reaches P8.46 (Pin_46)
- net AUX1: now also J4.3 (Pin_3)
- new net: L1.1, R21.2, U6.10 (SW)
- new net: C7.2, U6.3 (VINA)
- new net: R22.2, R23.1, U6.5 (FB)
- new net: R19.1, U6.6 (COMP)
- new net: C8.2, R18.1, U6.7 (EN_SS)
- new net: C10.2, U6.9 (BST)
- new net: C10.1, R21.1
- new net: C9.2, R19.2
- new net: R4.1, U1.1 (OUT0)
- new net: R6.1, U1.18 (OUT1)
- new net: R5.1, R7.1, U2.1, U2.2 (-)
- new net: R7.2, R9.1, U3.6 (-)
- new net: R11.1, R6.2, U3.5 (+)
- new net: J3.3 (Pin_3), R11.2, R13.1, U3.7
- new net: J3.1 (Pin_1), R17.2, U3.8
- new net: R13.2, R17.1, U3.9 (-)
- new net: R10.1, R4.2, U2.5 (+)
- new net: R5.2, R8.1, U2.6 (-)
- new net: J2.3 (Pin_3), R10.2, R12.1, U2.7
- new net: J2.1 (Pin_1), R16.2, U2.8
- new net: R12.2, R16.1, U2.9 (-)
- new net +15V: C3.2, C6.2, J1.3 (Pin_3), U2.4 (V+), U3.4 (V+), U5.1 (VIN), U5.4 (~SHDN), U6.2 (VINSW)
- new net +5VA: C2.2, C5.2, U1.16 (M/~Z), U1.24 (AVDD), U5.5 (VOUT)
- new net -15V: J1.1 (Pin_1), U2.11 (V-), U3.11 (V-)
Other:
- moved on the sheet: C4, P8, P9, R1, R14, R15, R2, R3, SW1, U4
