File: hardware/cape/_autosave-holobone.sch (KiCad schematic (older format))
At the start: 64 parts, among them J1 Conn_01x03, J3 Conn_01x03, J4 Conn_01x03, P1 BeagleBone_Black_Header, P2 BeagleBone_Black_Header, SW1 SW_DIP_x02, U1 LM4040DBZ-2.0, U2 CAT24C256, U3 TL084, U4 TL084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

Commit message: pcb prodiction
Parts:
- R10: Store https://uk.farnell.com/vishay/crcw080516k9fkea/res-16k9-1-0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 -> https://uk.farnell.com/vishay/crcw08052k00fkea/res-2k-1-0-1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
- R14: Store https://uk.farnell.com/vishay/crcw080516k9fkea/res-16k9-1-0-125w-0805-thick-film/dp/1652926RL -> https://uk.farnell.com/vishay/crcw080516k9fkea/res-16k9-1-0-125w-0805-thick-film/dp/1652926
Changed lines of the file:
@@
 F 2 "Resistor_SMD:R_0805_2012Metric" V 8280 4050 50  0001 C CNN
 F 3 "http://www.farnell.com/datasheets/2310790.pdf" H 8350 4050 50  0001 C CNN
-F 4 "https://uk.farnell.com/vishay/crcw080516k9fkea/res-16k9-1-0-125w-0805-thick-film/dp/1652926RL" H 8350 4050 50  0001 C CNN "Store"
+F 4 "https://uk.farnell.com/vishay/crcw080516k9fkea/res-16k9-1-0-125w-0805-thick-film/dp/1652926" H 8350 4050 50  0001 C CNN "Store"
 	1    8350 4050
 	1    0    0    -1
@@
 F 2 "Resistor_SMD:R_0805_2012Metric" V 2330 3000 50  0001 C CNN
 F 3 "http://www.farnell.com/datasheets/2310790.pdf" H 2400 3000 50  0001 C CNN
-F 4 "https://uk.farnell.com/vishay/crcw080516k9fkea/res-16k9-1-0-125w-0805-thick-film/dp/1652926RL" H 2400 3000 50  0001 C CNN "Store"
+F 4 "https://uk.farnell.com/vishay/crcw08052k00fkea/res-2k-1-0-125w-0805-thick-film/dp/1469884" H 2400 3000 50  0001 C CNN "Store"
 	1    2400 3000
 	1    0    0    -1
